File: ITR-3/ITR-3.kicad_sch (KiCad schematic)
At the start: 15 parts

Commit message: обновлена схема - добавлен буферный входной ОУ
Parts:
- added C1, C2, C3, C4: Конденсатор*0,1мкФ*25В*0603, N_RLC:Конденсатор_SMD_IEC_0603, symbol eo-engine:Конденсатор*0,1мкФ*25В*0603
- added DA2: ОУ_LMx58, N_DD:SO-8, symbol elements:ОУ_LMx58
- added R10, R11, R12, R4, R5, R6, R9: Резистор_0,065Вт, N_RLC:Резистор_SMD_0603_0,065_Вт, symbol elements:Резистор_0,065Вт
- added VD3, VD4: Диоды_шоттки_BAT54S, N_VD_HL:Транзистор_IRLML6344TR_SOT-23, symbol elements:Диоды_шоттки_BAT54S
- added VD5, VD6: Стабилитрон_1N5352BRLG_вертикальный, N_VD_HL:SOD-80, symbol elements_2020:Стабилитрон_1N5352BRLG_вертикальный
- added X1: Вилка_PLS3, N_X:Вилка_PLS3_вертикальная, symbol elements:Вилка_PLS3
- added X2: Вилка_PLS4, N_X:Вилка_PLS4_вертикальная, symbol elements:Вилка_PLS4
- R1: Номинал 100 Ом -> 470 Ом
- R2: Номинал 100 Ом -> 1 кОм
- R7: renamed from R4; Номинал 100 Ом -> 470 Ом
- R8: renamed from R5; Номинал 100 Ом -> 1 кОм
- renumbered DA2 to DA1, DA1 to DA3
Connections:
- net TXA is gone; now on net DA-B: R7.1, R8.1
- net TXB is gone; now on net DA-A: R1.2, R2.2
- net 5V: now also DA1.8 (VCC+), DA3.8 (VCC+), C1.1, C2.1, C4.1, DA2.8 (VCC+), R10.1, R9.1, VD3.2, VD4.2, X2.1
- net GND: now also DA1.4 (-VCC), DA3.4 (-VCC), C1.2, C2.2, C3.2, C4.2, DA2.4 (-VCC), R12.2, R4.1, VD3.1, VD4.1, VD5.1, VD6.1, X2.4
- net RSA: now also DA3.3, VD3.3, X2.3
- net RSB: now also DA3.5, VD4.3, X2.2
- net at VT3.2, VT5.2: now also R5.2; no longer VT2.3
- net DA-A: now reaches DA1.1
- net TX-OUT: now reaches DA1.2
- net TX-OUT: now also DA1.5, X1.1
- net AREF: now reaches DA1.3
- net AREF: now also DA1.6, C3.1, R11.2, R12.1
- net DA-B: now reaches DA1.7
- net RSEN: now reaches VT1.1
- net RSEN: now also R4.2, X1.2
- net at R3.1, VT4.2, VT6.2: now also R6.1; no longer VT1.3
- net at DA3.1: now also DA3.2
- net at DA3.6: now also DA3.7
- new net: R9.2, VD5.2
- new net: R5.1, VT2.3
- new net: R10.2, R11.1, VD6.2
- new net: R6.2, VT1.3
- new net RX-IN: X1.3
Other:
- moved on the sheet: DA1, DA3, R1, R2, R3, R7, R8, VD1, VD2, VT1, VT3, VT4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

Commit message: подготовлена трассировка и GBR для заказа
Parts:
- removed C1, C2, C4: Конденсатор*0,1мкФ*25В*0603, N_RLC:Конденсатор_SMD_IEC_0603, symbol eo-engine:Конденсатор*0,1мкФ*25В*0603
- removed DA1, DA2, DA3: ОУ_LMx58, N_DD:SO-8, symbol elements:ОУ_LMx58
- removed R1, R10, R11, R12, R2, R3, R5, R6, R7, R8, R9: Резистор_0,065Вт, N_RLC:Резистор_SMD_0603_0,065_Вт, symbol elements:Резистор_0,065Вт
- removed VD1, VD2, VD5, VD6: Стабилитрон_1N5352BRLG_вертикальный, N_VD_HL:SOD-80, symbol elements_2020:Стабилитрон_1N5352BRLG_вертикальный
- removed X1: Вилка_PLS3, N_X:Вилка_PLS3_вертикальная, symbol elements:Вилка_PLS3
- added C1, C2, C3: Конденсатор*0,1мкФ*25В*0603, KICAD6_RLC:Конденсатор_SMD_IEC_0603, symbol niisk_lib_C:smd-конденсатор-керамика*0,01мк*50В*0603*ВП
- added DA1, DA2, DA3: ОУ*сдвоенный*so-8*ОТК, MOTOR_IMPORT_OTK:SO-8, symbol niisk_lib:ОУ*сдвоенный*so-8*ОТК
- added R1, R4: smd-резистор*100к*0603*ВП, MOTOR_RLC:Резистор_SMD_IEC_0603-0,075_Вт, symbol niisk_lib:smd-резистор*100к*0603*ВП
- added R10, R13, R9: smd-резистор*4,7*0,1Вт*5проц*0603*ВП, KICAD6_RLC:Резистор_SMD_IEC_0603-0,1_Вт, symbol niisk_lib_R:smd-резистор*4,7*0,1Вт*5проц*0603*ВП
- added R11, R2: smd-резистор*470*0,1Вт*5проц*0603*ВП, KICAD6_RLC:Резистор_SMD_IEC_0603-0,1_Вт, symbol niisk_lib_R:smd-резистор*470*0,1Вт*5проц*0603*ВП
- added R12, R14, R3, R5: smd-резистор*1к*0,1Вт*5проц*0603*ВП, KICAD6_RLC:Резистор_SMD_IEC_0603-0,1_Вт, symbol niisk_lib_R:smd-резистор*1к*0,1Вт*5проц*0603*ВП
- added R15, R16: smd-резистор*10к*0,1Вт*5проц*0603*ВП, KICAD6_RLC:Резистор_SMD_IEC_0603-0,1_Вт, symbol niisk_lib_R:smd-резистор*10к*0,1Вт*5проц*0603*ВП
- added R6, R7: smd-резистор*20к*0603*ВП, MOTOR_RLC:Резистор_SMD_IEC_0603-0,075_Вт, symbol niisk_lib:smd-резистор*20к*0603*ВП
- added VD1, VD2, VD5, VD6: smd-стабилитрон*5,1В*5мА*КД-36*ВП, MOTOR_VD_VT_HL:Корпус_IEC_КД-36, symbol niisk_lib:smd-стабилитрон*5,1В*5мА*КД-36*ВП
- added XP1: Вилка*PLS*3контакта*1ряд*вертикальная, MOTOR_X:Вилка_SNP346-3VP21-1, symbol niisk_lib:Вилка*PLS*3контакта*1ряд*вертикальная
- C4: renamed from C3; footprint N_RLC:Конденсатор_SMD_IEC_0603 -> KICAD6_RLC:Конденсатор_SMD_IEC_0603; symbol eo-engine:Конденсатор*0,1мкФ*25В*0603 -> niisk_lib_C:smd-конденсатор-керамика*0,01мк*50В*0603*ВП; INFO 0,1мкФ 25В -> 0,01мк 50В; NAME (none) -> Конденсатор К10-79-50В-0,01мкФ+80-20проц.-Н90 АЖЯР.673511.0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; SUPPLIER (none) -> ООО "Кулон", г. Санкт-Петербург; SYMBOL (none) -> 2.728; ЭКБ (none) -> 2021
- VD3, VD4: footprint N_VD_HL:Транзистор_IRLML6344TR_SOT-23 -> MOTOR_VD_VT_HL:Корпус_КТ-46
- renumbered R4 to R8, X2 to X1
Connections:
- net 5V: now also C1.2, C2.2, C3.2, DA1.8, DA2.8, DA3.8, R13.2, R14.2
- net AREF: now also C4.2, DA1.3, DA1.6, DA2.2, R15.1, R16.2; no longer C4.1
- net DA-A: now also DA1.1, R2.1, R3.2
- net DA-B: now also DA1.7, R11.2, R12.1
- net GND: now also C4.1, C1.1, C2.1, C3.1, DA1.4, DA2.4, DA3.4, R16.1, R4.1, VD5.A, VD6.A; no longer C4.2
- net RSA: now also DA3.3
- net RSB: now also DA3.5
- net RSEN: now also XP1.2A
- net RX-IN: now also DA2.1, XP1.3A
- net TX-OUT: now also DA1.2, DA1.5, XP1.1A
- net at VT3.1: now also VD1.K
- net at VT3.2, VT5.2: now also R9.1
- net at VT6.1: now also R12.2
- net at VT2.3: now also R9.2
- net at VT1.3: now also R10.1, R5.1
- net at VT4.2, VT6.2: now also R10.2
- net at VT4.1: now also R3.1
- net at VT5.1: now also VD2.K
- net at VT2.1: now also R5.2
- new net: R11.1, VD2.A
- new net: DA2.3, DA2.7, R1.1
- new net: DA2.5, R4.2, R7.1
- new net: DA2.6, R1.2, R6.1
- new net: R13.1, VD5.K
- new net: R14.1, R15.2, VD6.K
- new net: R2.2, VD1.A
- new net BUFA: DA3.1, DA3.2, R7.2
- new net BUFB: DA3.6, DA3.7, R6.2
Other:
- moved on the sheet: C4, R8, VD3, VD4, VT1, VT2, VT3, VT4, VT5, VT6, X1
